Commit message: added satellite model

File: src/space_panda_description/space_panda_description/urdf/space_panda.urdf.xacro (robot description, xacro)
@@ -6,16 +6,21 @@
   <xacro:property name="load_gripper" value="true"/>
   <xacro:property name="ee_id" value="franka_hand"/>
+  <!-- World frame to anchor the satellite + robot system -->
+  <link name="world"/>
+  <!-- Satellite body (realistic mesh) the robot will sit on -->
+  <!-- Uses cubesat mesh from the package's meshes directory -->
   <link name="satellite_base">
     <visual>
       <geometry>
-        <box size="1 1 0.5"/>
+        <mesh filename="package://space_panda_description/meshes/cubesat.stl" scale="0.5 0.5 0.5"/>
       </geometry>
-      <material name="grey">
+      <material name="satellite_grey">
         <color rgba="0.6 0.6 0.6 1.0"/>
       </material>
     </visual>
+    <!-- Use same mesh for collision for now; you can swap to a simplified collision mesh later -->
     <collision>
       <geometry>
-        <box size="1 1 0.5"/>
+        <mesh filename="package://space_panda_description/meshes/cubesat.stl" scale="0.5 0.5 0.5"/>
       </geometry>
     </collision>
@@ -29,7 +34,15 @@
     </inertial>
   </link>
+  <!-- Fix the satellite in the world frame -->
+  <joint name="world_to_satellite" type="fixed">
+    <origin xyz="0 0 0" rpy="0 0 0"/>
+    <parent link="world"/>
+    <child link="satellite_base"/>
+  </joint>
   <!-- Joint between satellite and Franka base -->
+  <!-- Increase z so the robot base sits on top of the satellite mesh, not inside it -->
   <joint name="satellite_to_franka" type="fixed">
-    <origin xyz="0 0 0.25" rpy="0 0 0"/>
+    <!-- Tune this z value based on your cubesat mesh thickness (start with 0.5) -->
+    <origin xyz="0 0 0.75" rpy="0 0 0"/>
     <parent link="satellite_base"/>
     <child link="fr3_link0"/>

Commit message: added cubesat

File: src/space_panda_description/space_panda_description/urdf/space_panda.urdf.xacro (robot description, xacro)
@@ -9,9 +9,12 @@
   <link name="world"/>
   <!-- Satellite body (realistic mesh) the robot will sit on -->
-  <!-- Uses cubesat mesh from the package's meshes directory -->
+  <!-- Uses cubesat mesh from the package's meshes directory.
+       Use an absolute file:// URI so Gazebo can always resolve it. -->
   <link name="satellite_base">
     <visual>
       <geometry>
-        <mesh filename="package://space_panda_description/meshes/cubesat.stl" scale="0.5 0.5 0.5"/>
+        <mesh
+          filename="file:///home/anish/data/SpaceTS/robotics/space_robotics/src/space_panda_description/meshes/cubesat.stl"
+          scale="0.5 0.5 0.5"/>
       </geometry>
       <material name="satellite_grey">
@@ -22,5 +25,7 @@
     <collision>
       <geometry>
-        <mesh filename="package://space_panda_description/meshes/cubesat.stl" scale="0.5 0.5 0.5"/>
+        <mesh
+          filename="file:///home/anish/data/SpaceTS/robotics/space_robotics/src/space_panda_description/meshes/cubesat.stl"
+          scale="0.5 0.5 0.5"/>
       </geometry>
     </collision>

Commit message: gazebo

File: src/space_panda_description/space_panda_description/urdf/space_panda.urdf.xacro (robot description, xacro)
@@ -1,19 +1,16 @@
 <?xml version="1.0"?>
 <robot name="space_panda" xmlns:xacro="http://www.ros.org/wiki/xacro">
-  <!-- Load generic Franka robot macro -->
+  <!-- ✅ ROS 2 SAFE INCLUDE -->
   <xacro:include filename="$(find franka_description)/robots/common/franka_robot.xacro"/>
-  <!-- Parameters -->
   <xacro:property name="load_gripper" value="true"/>
   <xacro:property name="ee_id" value="franka_hand"/>
-  <!-- World frame to anchor the satellite + robot system -->
+  <!-- ================= WORLD ================= -->
   <link name="world"/>
-  <!-- Satellite body (realistic mesh) the robot will sit on -->
-  <!-- Uses cubesat mesh from the package's meshes directory.
-       Use an absolute file:// URI so Gazebo can always resolve it. -->
+  <!-- ================= SATELLITE ================= -->
   <link name="satellite_base">
     <visual>
       <geometry>
         <mesh
-          filename="file:///home/anish/data/SpaceTS/robotics/space_robotics/src/space_panda_description/meshes/cubesat.stl"
+          filename="$(find space_panda_description)/meshes/cubesat.stl"
           scale="0.5 0.5 0.5"/>
       </geometry>
@@ -22,11 +19,10 @@
       </material>
     </visual>
-    <!-- Use same mesh for collision for now; you can swap to a simplified collision mesh later -->
+    <!-- ✅ SIMPLE collision for stable physics -->
     <collision>
       <geometry>
-        <mesh
-          filename="file:///home/anish/data/SpaceTS/robotics/space_robotics/src/space_panda_description/meshes/cubesat.stl"
-          scale="0.5 0.5 0.5"/>
+        <box size="0 0 0"/>
       </geometry>
+      <origin xyz="1.4 1.4 1.2"/>
     </collision>
     <inertial>
@@ -39,18 +35,19 @@
     </inertial>
   </link>
-  <!-- Fix the satellite in the world frame -->
+  <!-- World → Satellite -->
+  <gazebo reference="satellite_base">
+    <static>true</static>
+  </gazebo>
   <joint name="world_to_satellite" type="fixed">
-    <origin xyz="0 0 0" rpy="0 0 0"/>
     <parent link="world"/>
     <child link="satellite_base"/>
   </joint>
-  <!-- Joint between satellite and Franka base -->
-  <!-- Increase z so the robot base sits on top of the satellite mesh, not inside it -->
+  <!-- ================= FR3 ROBOT ================= -->
   <joint name="satellite_to_franka" type="fixed">
-    <!-- Tune this z value based on your cubesat mesh thickness (start with 0.5) -->
     <origin xyz="0 0 0.75" rpy="0 0 0"/>
     <parent link="satellite_base"/>
     <child link="fr3_link0"/>
   </joint>
+  <!-- ✅ ROS 2 SAFE YAML LOADS -->
   <xacro:franka_robot
     arm_id="fr3"
@@ -62,4 +59,56 @@
     hand="${load_gripper}"
     ee_id="${ee_id}"
-    connected_to=""/>
+    connected_to=""
+  />
+  <!-- ================= ROS2 CONTROL ================= -->
+  <ros2_control name="FR3System" type="system">
+    <hardware>
+      <plugin>gazebo_ros2_control/GazeboSystem</plugin>
+    </hardware>
+    <!-- Arm joints -->
+    <joint name="fr3_joint1">
+      <command_interface name="position"/>
+      <state_interface name="position"/>
+      <state_interface name="velocity"/>
+    </joint>
+    <joint name="fr3_joint2">
+      <command_interface name="position"/>
+      <state_interface name="position"/>
+      <state_interface name="velocity"/>
+    </joint>
+    <joint name="fr3_joint3">
+      <command_interface name="position"/>
+      <state_interface name="position"/>
+      <state_interface name="velocity"/>
+    </joint>
+    <joint name="fr3_joint4">
+      <command_interface name="position"/>
+      <state_interface name="position"/>
+      <state_interface name="velocity"/>
+    </joint>
+    <joint name="fr3_joint5">
+      <command_interface name="position"/>
+      <state_interface name="position"/>
+      <state_interface name="velocity"/>
+    </joint>
+    <joint name="fr3_joint6">
+      <command_interface name="position"/>
+      <state_interface name="position"/>
+      <state_interface name="velocity"/>
+    </joint>
+    <joint name="fr3_joint7">
+      <command_interface name="position"/>
+      <state_interface name="position"/>
+      <state_interface name="velocity"/>
+    </joint>
+    <!-- ✅ GRIPPER (FIXED MIMIC BUG) -->
+    <joint name="fr3_finger_joint1">
+      <command_interface name="position"/>
+      <state_interface name="position"/>
+    </joint>
+    <!-- ✅ Mimic joint MUST NOT have command interface -->
+    <joint name="fr3_finger_joint2">
+      <state_interface name="position"/>
+    </joint>
+  </ros2_control>
 </robot>

Commit message: adding space world

File: src/space_panda_description/space_panda_description/urdf/space_panda.urdf.xacro (robot description, xacro)
@@ -22,7 +22,9 @@
     <collision>
       <geometry>
-        <box size="0 0 0"/>
+        <!-- 1.5m box to match roughly with the visual scale and arm mounting height -->
+        <box size="1.5 1.5 1.5"/>
       </geometry>
-      <origin xyz="1.4 1.4 1.2"/>
+      <!-- Center the collision box -->
+      <origin xyz="0 0 0"/>
     </collision>
     <inertial>

Commit message: panda movement

File: src/space_panda_description/space_panda_description/urdf/space_panda.urdf.xacro (robot description, xacro)
@@ -5,7 +5,6 @@
   <xacro:property name="load_gripper" value="true"/>
   <xacro:property name="ee_id" value="franka_hand"/>
-  <!-- ================= WORLD ================= -->
-  <link name="world"/>
-  <!-- ================= SATELLITE ================= -->
+  <!-- ================= SATELLITE BASE (ROOT LINK) ================= -->
+  <!-- No world link needed - satellite_base is the root, allowing free motion in space -->
   <link name="satellite_base">
     <visual>
@@ -37,12 +36,8 @@
     </inertial>
   </link>
-  <!-- World → Satellite -->
+  <!-- Satellite is dynamic (can move freely in space) -->
   <gazebo reference="satellite_base">
-    <static>true</static>
-  </gazebo>
-  <joint name="world_to_satellite" type="fixed">
-    <parent link="world"/>
-    <child link="satellite_base"/>
-  </joint>
+    <static>false</static>
+  </gazebo>
   <!-- ================= FR3 ROBOT ================= -->
   <joint name="satellite_to_franka" type="fixed">
@@ -63,54 +58,213 @@
     connected_to=""
   />
-  <!-- ================= ROS2 CONTROL ================= -->
-  <ros2_control name="FR3System" type="system">
-    <hardware>
-      <plugin>gazebo_ros2_control/GazeboSystem</plugin>
-    </hardware>
-    <!-- Arm joints -->
-    <joint name="fr3_joint1">
-      <command_interface name="position"/>
-      <state_interface name="position"/>
-      <state_interface name="velocity"/>
-    </joint>
-    <joint name="fr3_joint2">
-      <command_interface name="position"/>
-      <state_interface name="position"/>
-      <state_interface name="velocity"/>
-    </joint>
-    <joint name="fr3_joint3">
-      <command_interface name="position"/>
-      <state_interface name="position"/>
-      <state_interface name="velocity"/>
-    </joint>
-    <joint name="fr3_joint4">
-      <command_interface name="position"/>
-      <state_interface name="position"/>
-      <state_interface name="velocity"/>
-    </joint>
-    <joint name="fr3_joint5">
-      <command_interface name="position"/>
-      <state_interface name="position"/>
-      <state_interface name="velocity"/>
-    </joint>
-    <joint name="fr3_joint6">
-      <command_interface name="position"/>
-      <state_interface name="position"/>
-      <state_interface name="velocity"/>
-    </joint>
-    <joint name="fr3_joint7">
-      <command_interface name="position"/>
-      <state_interface name="position"/>
-      <state_interface name="velocity"/>
-    </joint>
-    <!-- ✅ GRIPPER (FIXED MIMIC BUG) -->
-    <joint name="fr3_finger_joint1">
-      <command_interface name="position"/>
-      <state_interface name="position"/>
-    </joint>
-    <!-- ✅ Mimic joint MUST NOT have command interface -->
-    <joint name="fr3_finger_joint2">
-      <state_interface name="position"/>
-    </joint>
-  </ros2_control>
+  <!-- ================= GAZEBO PLUGINS FOR CONTROL ================= -->
+  <!-- Odometry Publisher for Satellite -->
+  <gazebo>
+    <plugin name="odometry_publisher" filename="gz-sim-odometry-publisher-system">
+      <dimensions>3</dimensions>
+      <odom_publish_frequency>50.0</odom_publish_frequency>
+      <odom_frame>world</odom_frame>
+      <robot_base_frame>satellite_base</robot_base_frame>
+    </plugin>
+  </gazebo>
+  <!-- Joint Position Controllers for FR3 Arm -->
+  <gazebo>
+    <plugin filename="gz-sim-joint-position-controller-system"
+            name="gz::sim::systems::JointPositionController">
+      <joint_name>fr3_joint1</joint_name>
+      <topic>fr3/joint1_cmd</topic>
+      <p_gain>100</p_gain>
+      <i_gain>10</i_gain>
+      <d_gain>5</d_gain>
+      <i_max>10</i_max>
+      <i_min>-10</i_min>
+      <cmd_max>2.8973</cmd_max>
+      <cmd_min>-2.8973</cmd_min>
+    </plugin>
+  </gazebo>
+  <gazebo>
+    <plugin filename="gz-sim-joint-position-controller-system"
+            name="gz::sim::systems::JointPositionController">
+      <joint_name>fr3_joint2</joint_name>
+      <topic>fr3/joint2_cmd</topic>
+      <p_gain>100</p_gain>
+      <i_gain>10</i_gain>
+      <d_gain>5</d_gain>
+      <i_max>10</i_max>
+      <i_min>-10</i_min>
+      <cmd_max>1.7628</cmd_max>
+      <cmd_min>-1.7628</cmd_min>
+    </plugin>
+  </gazebo>
+  <gazebo>
+    <plugin filename="gz-sim-joint-position-controller-system"
+            name="gz::sim::systems::JointPositionController">
+      <joint_name>fr3_joint3</joint_name>
+      <topic>fr3/joint3_cmd</topic>
+      <p_gain>100</p_gain>
+      <i_gain>10</i_gain>
+      <d_gain>5</d_gain>
+      <i_max>10</i_max>
+      <i_min>-10</i_min>
+      <cmd_max>2.8973</cmd_max>
+      <cmd_min>-2.8973</cmd_min>
+    </plugin>
+  </gazebo>
+  <gazebo>
+    <plugin filename="gz-sim-joint-position-controller-system"
+            name="gz::sim::systems::JointPositionController">
+      <joint_name>fr3_joint4</joint_name>
+      <topic>fr3/joint4_cmd</topic>
+      <p_gain>100</p_gain>
+      <i_gain>10</i_gain>
+      <d_gain>5</d_gain>
+      <i_max>10</i_max>
+      <i_min>-10</i_min>
+      <cmd_max>-0.0698</cmd_max>
+      <cmd_min>-3.0718</cmd_min>
+    </plugin>
+  </gazebo>
+  <gazebo>
+    <plugin filename="gz-sim-joint-position-controller-system"
+            name="gz::sim::systems::JointPositionController">
+      <joint_name>fr3_joint5</joint_name>
+      <topic>fr3/joint5_cmd</topic>
+      <p_gain>100</p_gain>
+      <i_gain>10</i_gain>
+      <d_gain>5</d_gain>
+      <i_max>10</i_max>
+      <i_min>-10</i_min>
+      <cmd_max>2.8973</cmd_max>
+      <cmd_min>-2.8973</cmd_min>
+    </plugin>
+  </gazebo>
+  <gazebo>
+    <plugin filename="gz-sim-joint-position-controller-system"
+            name="gz::sim::systems::JointPositionController">
+      <joint_name>fr3_joint6</joint_name>
+      <topic>fr3/joint6_cmd</topic>
+      <p_gain>100</p_gain>
+      <i_gain>10</i_gain>
+      <d_gain>5</d_gain>
+      <i_max>10</i_max>
+      <i_min>-10</i_min>
+      <cmd_max>3.7525</cmd_max>
+      <cmd_min>-0.0175</cmd_min>
+    </plugin>
+  </gazebo>
+  <gazebo>
+    <plugin filename="gz-sim-joint-position-controller-system"
+            name="gz::sim::systems::JointPositionController">
+      <joint_name>fr3_joint7</joint_name>
+      <topic>fr3/joint7_cmd</topic>
+      <p_gain>100</p_gain>
+      <i_gain>10</i_gain>
+      <d_gain>5</d_gain>
+      <i_max>10</i_max>
+      <i_min>-10</i_min>
+      <cmd_max>2.8973</cmd_max>
+      <cmd_min>-2.8973</cmd_min>
+    </plugin>
+  </gazebo>
+  <!-- Gripper Controllers -->
+  <gazebo>
+    <plugin filename="gz-sim-joint-position-controller-system"
+            name="gz::sim::systems::JointPositionController">
+      <joint_name>fr3_finger_joint1</joint_name>
+      <topic>fr3/gripper_cmd</topic>
+      <p_gain>50</p_gain>
+      <i_gain>5</i_gain>
+      <d_gain>1</d_gain>
+      <i_max>5</i_max>
+      <i_min>-5</i_min>
+      <cmd_max>0.04</cmd_max>
+      <cmd_min>0.0</cmd_min>
+    </plugin>
+  </gazebo>
+  <!-- Thrusters for orbital adjustments -->
+  <link name="forward_thruster">
+    <inertial>
+      <mass value="0.01"/>
+      <origin xyz="0 0 0"/>
+      <inertia
+        ixx="0.0001" ixy="0" ixz="0"
+        iyy="0.0001" iyz="0"
+        izz="0.0001"/>
+    </inertial>
+  </link>
+  <joint name="forward_thruster_joint" type="revolute">
+    <parent link="satellite_base"/>
+    <child link="forward_thruster"/>
+    <origin xyz="0 0 0"/>
+    <axis xyz="1 0 0"/>
+    <limit lower="-1e16" upper="1e16" effort="1000" velocity="1000"/>
+  </joint>
+  <link name="lateral_thruster">
+    <inertial>
+      <mass value="0.01"/>
+      <origin xyz="0 0 0"/>
+      <inertia
+        ixx="0.0001" ixy="0" ixz="0"
+        iyy="0.0001" iyz="0"
+        izz="0.0001"/>
+    </inertial>
+  </link>
+  <joint name="lateral_thruster_joint" type="revolute">
+    <parent link="satellite_base"/>
+    <child link="lateral_thruster"/>
+    <origin xyz="0 0 0"/>
+    <axis xyz="0 1 0"/>
+    <limit lower="-1e16" upper="1e16" effort="1000" velocity="1000"/>
+  </joint>
+  <link name="vertical_thruster">
+    <inertial>
+      <mass value="0.01"/>
+      <origin xyz="0 0 0"/>
+      <inertia
+        ixx="0.0001" ixy="0" ixz="0"
+        iyy="0.0001" iyz="0"
+        izz="0.0001"/>
+    </inertial>
+  </link>
+  <joint name="vertical_thruster_joint" type="revolute">
+    <parent link="satellite_base"/>
+    <child link="vertical_thruster"/>
+    <origin xyz="0 0 0"/>
+    <axis xyz="0 0 1"/>
+    <limit lower="-1e16" upper="1e16" effort="1000" velocity="1000"/>
+  </joint>
+  <!-- Thruster Plugins -->
+  <gazebo>
+    <plugin filename="gz-sim-thruster-system"
+            name="gz::sim::systems::Thruster">
+      <joint_name>forward_thruster_joint</joint_name>
+      <thrust_coefficient>0.01</thrust_coefficient>
+      <fluid_density>1.0</fluid_density>
+      <propeller_diameter>0.5</propeller_diameter>
+      <max_thrust_cmd>100</max_thrust_cmd>
+      <min_thrust_cmd>-100</min_thrust_cmd>
+    </plugin>
+  </gazebo>
+  <gazebo>
+    <plugin filename="gz-sim-thruster-system"
+            name="gz::sim::systems::Thruster">
+      <joint_name>lateral_thruster_joint</joint_name>
+      <thrust_coefficient>0.01</thrust_coefficient>
+      <fluid_density>1.0</fluid_density>
+      <propeller_diameter>0.5</propeller_diameter>
+      <max_thrust_cmd>100</max_thrust_cmd>
+      <min_thrust_cmd>-100</min_thrust_cmd>
+    </plugin>
+  </gazebo>
+  <gazebo>
+    <plugin filename="gz-sim-thruster-system"
+            name="gz::sim::systems::Thruster">
+      <joint_name>vertical_thruster_joint</joint_name>
+      <thrust_coefficient>0.01</thrust_coefficient>
+      <fluid_density>1.0</fluid_density>
+      <propeller_diameter>0.5</propeller_diameter>
+      <max_thrust_cmd>100</max_thrust_cmd>
+      <min_thrust_cmd>-100</min_thrust_cmd>
+    </plugin>
+  </gazebo>
 </robot>
