Commit message: dynamic cam with gui

File: src/space_panda_description/space_panda_description/urdf/space_panda.urdf.xacro (robot description, xacro)
@@ -39,21 +39,94 @@
   <gazebo reference="satellite_base">
     <static>false</static>
-    <!-- Camera sensor to view arm/gripper and Earth -->
+  </gazebo>
+  <!-- ================= PAN-TILT CAMERA SYSTEM ================= -->
+  <!-- Camera Base (for azimuth rotation) -->
+  <link name="camera_base">
+    <inertial>
+      <mass value="0.1"/>
+      <origin xyz="0 0 0"/>
+      <inertia
+        ixx="0.001" ixy="0" ixz="0"
+        iyy="0.001" iyz="0"
+        izz="0.001"/>
+    </inertial>
+    <visual>
+      <geometry>
+        <cylinder radius="0.05" length="0.1"/>
+      </geometry>
+      <material name="camera_mount">
+        <color rgba="0.3 0.3 0.3 1.0"/>
+      </material>
+    </visual>
+  </link>
+  <!-- Joint: Satellite → Camera Base (Azimuth/Horizontal rotation) -->
+  <joint name="camera_azimuth_joint" type="revolute">
+    <parent link="satellite_base"/>
+    <child link="camera_base"/>
+    <origin xyz="0 0 1.0" rpy="0 0 0"/>  <!-- Mount on top of satellite -->
+    <axis xyz="0 0 1"/>  <!-- Rotate around Z axis (horizontal spin) -->
+    <limit lower="-6.28319" upper="6.28319" effort="10" velocity="1.0"/>  <!-- 360° rotation -->
+  </joint>
+  <!-- Camera Tilt Mount (for elevation) -->
+  <link name="camera_tilt">
+    <inertial>
+      <mass value="0.05"/>
+      <origin xyz="0 0 0"/>
+      <inertia
+        ixx="0.0005" ixy="0" ixz="0"
+        iyy="0.0005" iyz="0"
+        izz="0.0005"/>
+    </inertial>
+    <visual>
+      <geometry>
+        <box size="0.08 0.05 0.05"/>
+      </geometry>
+      <material name="camera_tilt">
+        <color rgba="0.2 0.2 0.2 1.0"/>
+      </material>
+    </visual>
+  </link>
+  <!-- Joint: Camera Base → Camera Tilt (Elevation/Vertical tilt) -->
+  <joint name="camera_elevation_joint" type="revolute">
+    <parent link="camera_base"/>
+    <child link="camera_tilt"/>
+    <origin xyz="0 0 0.05" rpy="0 0 0"/>
+    <axis xyz="0 1 0"/>  <!-- Rotate around Y axis (tilt up/down) -->
+    <limit lower="-3.14159" upper="3.14159" effort="10" velocity="1.0"/>  <!-- 180° up/down -->
+  </joint>
+  <!-- Camera Link (actual camera sensor) -->
+  <link name="camera_link">
+    <inertial>
+      <mass value="0.02"/>
+      <origin xyz="0 0 0"/>
+      <inertia
+        ixx="0.0001" ixy="0" ixz="0"
+        iyy="0.0001" iyz="0"
+        izz="0.0001"/>
+    </inertial>
+    <visual>
+      <geometry>
+        <box size="0.03 0.06 0.03"/>
+      </geometry>
+      <material name="camera_body">
+        <color rgba="0.1 0.1 0.1 1.0"/>
+      </material>
+    </visual>
+  </link>
+  <!-- Joint: Camera Tilt → Camera (fixed) -->
+  <joint name="camera_optical_joint" type="fixed">
+    <parent link="camera_tilt"/>
+    <child link="camera_link"/>
+    <origin xyz="0.04 0 0" rpy="0 0 0"/>  <!-- Camera faces forward from tilt mount -->
+  </joint>
+  <!-- Camera Sensor -->
+  <gazebo reference="camera_link">
     <sensor name="satellite_camera" type="camera">
-      <!-- Position: Side-mounted to see arm clearly
-           Camera mounted to the SIDE of satellite
-           Looking across toward the arm with Earth as backdrop
-           X: -0.5m (back from center, away from Earth)
-           Y: -0.8m (to the side - left of arm)
-           Z: 0.9m (at mid-arm height)
-           Yaw: 0.5 rad (~30°) to look at arm from angle
-           Pitch: 0.1 rad (slight down angle)
-           This gives oblique view: arm in foreground, Earth in background -->
-      <pose>-0.5 -0.8 0.9 0 0.1 0.5</pose>  <!-- Side-angled view of arm -->
+      <pose>0 0 0 0 0 0</pose>  <!-- Camera faces in +X direction of camera_link -->
       <camera>
         <horizontal_fov>1.5708</horizontal_fov>  <!-- 90 degrees FOV -->
         <image>
-          <width>1280</width>
-          <height>720</height>
+          <width>640</width>
+          <height>480</height>
           <format>R8G8B8</format>
         </image>
@@ -69,8 +142,37 @@
       </camera>
       <always_on>1</always_on>
-      <update_rate>30</update_rate>
+      <update_rate>10</update_rate>
       <visualize>true</visualize>
       <topic>satellite_camera</topic>
     </sensor>
+  </gazebo>
+  <!-- Gazebo Plugins for Camera Control -->
+  <gazebo>
+    <plugin filename="gz-sim-joint-position-controller-system"
+            name="gz::sim::systems::JointPositionController">
+      <joint_name>camera_azimuth_joint</joint_name>
+      <topic>camera/azimuth_cmd</topic>
+      <p_gain>50</p_gain>
+      <i_gain>5</i_gain>
+      <d_gain>2</d_gain>
+      <i_max>5</i_max>
+      <i_min>-5</i_min>
+      <cmd_max>6.28319</cmd_max>
+      <cmd_min>-6.28319</cmd_min>
+    </plugin>
+  </gazebo>
+  <gazebo>
+    <plugin filename="gz-sim-joint-position-controller-system"
+            name="gz::sim::systems::JointPositionController">
+      <joint_name>camera_elevation_joint</joint_name>
+      <topic>camera/elevation_cmd</topic>
+      <p_gain>50</p_gain>
+      <i_gain>5</i_gain>
+      <d_gain>2</d_gain>
+      <i_max>5</i_max>
+      <i_min>-5</i_min>
+      <cmd_max>3.14159</cmd_max>
+      <cmd_min>-3.14159</cmd_min>
+    </plugin>
   </gazebo>
   <!-- ================= FR3 ROBOT ================= -->
